Commit message: feat: add go2.

File: legged_examples/legged_unitree/legged_unitree_description/urdf/robot.xacro (robot description, xacro)
@@ -8,5 +8,5 @@
     <xacro:include filename="$(find legged_unitree_description)/urdf/$(arg robot_type)/const.xacro"/>
 <!--    <xacro:property name="mesh_path" value="../meshes"/>-->
-    <xacro:property name="mesh_path" value="$(find legged_unitree_description)/meshes/$(arg robot_type)"/>
+    <xacro:property name="mesh_path" value="file://$(find legged_unitree_description)/meshes/$(arg robot_type)"/>
     <link name="base">
         <visual>
@@ -32,4 +32,5 @@
     </link>
     <xacro:IMU connected_to="base" imu_name="base_imu" xyz="0. 0. 0." rpy="0. 0. 0."/>
+    <!-- <xacro:IMU connected_to="base" imu_name="unitree_imu" xyz="0. 0. 0." rpy="0. 0. 0."/> -->
     <xacro:leg prefix="LF" mesh_path="${mesh_path}" mirror="1" mirror_dae="True" front_hind="1" front_hind_dae="True">
         <origin rpy="0 0 0" xyz="${leg_offset_x} ${leg_offset_y} 0"/>
